Commit message: ball attached to chain

File: jaco_gym/envs/assets/models/ball_and_cup/chain.urdf.xacro (robot description, xacro)
@@ -2,4 +2,5 @@
 <robot xmlns:xacro="http://www.ros.org/wiki/xacro" name="chain">
 	<xacro:property name="link_length" value="0.1" />
+	<xacro:property name="link_num" value="4"/>
 	<xacro:macro name="chain_link" params="name X Y Z mass">
 		<link name="${name}">
@@ -27,46 +28,37 @@
 			<origin xyz="${X} 0 0" rpy="0 0 0"/>
 			<parent link="${parent}"/>
-			<child link="junta1"/>
+			<child link="${name}_junta1"/>
 			<axis xyz="0 1 0" />
 		</joint>
-		<link name="junta1">
+		<link name="${name}_junta1">
 			<inertial>
-			<mass value="0.025" />
+			<mass value="0.001" />
 			<inertia ixx="5.8083e-4" ixy="0" ixz="0" iyy="3.0833e-5" iyz="0" izz="5.9083e-4" />
 			</inertial>
 		</link>
 		<joint name="${name}_joint2" type="continuous">
-			<parent link="junta1"/>
-			<child link="junta2"/>
+			<parent link="${name}_junta1"/>
+			<child link="${name}_junta2"/>
 			<axis xyz="0 0 1" />
 		</joint>
-		<link name="junta2">
+		<link name="${name}_junta2">
 			<inertial>
-			<mass value="0.025" />
+			<mass value="0.001" />
 			<inertia ixx="5.8083e-4" ixy="0" ixz="0" iyy="3.0833e-5" iyz="0" izz="5.9083e-4" />
 			</inertial>
 		</link>
 		<joint name="${name}_joint3" type="continuous">
-			<parent link="junta1"/>
-			<child link="junta3"/>
+			<parent link="${name}_junta1"/>
+			<child link="${name}_junta3"/>
 			<axis xyz="1 0 0" />
 		</joint>
-		<link name="junta3">
+		<link name="${name}_junta3">
 			<inertial>
-			<mass value="0.025" />
+			<mass value="0.001" />
 			<inertia ixx="5.8083e-4" ixy="0" ixz="0" iyy="3.0833e-5" iyz="0" izz="5.9083e-4" />
 			</inertial>
 		</link>
 		<joint name="${name}_jointfixed" type="fixed">
-			<parent link="junta3"/>
-			<child link="${name}"/>
-		</joint>
-	</xacro:macro>
-	<xacro:macro name="link_joint" params="name X parent">
-		<joint name="${name}_link_joint" type="continuous">
-			<!-- <dynamics damping="0.00001" friction="0.00001"/> -->
-			<origin xyz="${X} 0 0" rpy="0 0 0" />
-			<axis xyz="0 1 0" />
-			<parent link="${parent}"/>
+			<parent link="${name}_junta3"/>
 			<child link="${name}"/>
 		</joint>
@@ -85,27 +77,61 @@
 	  </gazebo>
 	</xacro:macro>
-	<link name="chain_base">
-	</link>
-	<xacro:chain_link name="0" X="${link_length}" Y="0.01" Z="0.01" mass="0.001"/>
-	<joint name="0" type="fixed">
-		<origin xyz="0 0 0" rpy="0 0 0" />
-		<parent link="chain_base"/>
-		<child link="0"/>
-	</joint>
-	<xacro:link_gazebo name="0" />
-	<xacro:chain_link name="1" X="${link_length}" Y="0.01" Z="0.01" mass="0.001"/>
-	<xacro:link_ball_joint name="1" X="${link_length}" parent="0"/>
-	<xacro:link_gazebo name="1"/>
-	<xacro:chain_link name="2" X="${link_length}" Y="0.01" Z="0.01" mass="0.001"/>
-	<xacro:link_ball_joint name="2" X="${link_length}" parent="1"/>
-	<xacro:link_gazebo name="2"/>
-	<xacro:chain_link name="3" X="${link_length}" Y="0.01" Z="0.01" mass="0.001"/>
-	<xacro:link_ball_joint name="3" X="${link_length}" parent="2"/>
-	<xacro:link_gazebo name="3"/>
-	<!-- <xacro:macro name="loop" params="links_qty">
-		<xacro:if value="${links_qty}">
-			<xacro:loop links_qty="${links_qty-1}" />
+	<xacro:macro name="chain_loop" params="i">
+		<xacro:chain_link name="${link_num - i + 1}" X="${link_length}" Y="0.01" Z="0.01" mass="0.001"/>
+		<xacro:link_ball_joint name="${link_num - i + 1}" X="${link_length}" parent="${link_num - i}"/>
+		<xacro:link_gazebo name="${link_num - i + 1}"/>
+		<xacro:if value="${i-1}">
+			<xacro:chain_loop i="${i-1}" />
 		</xacro:if>
 	</xacro:macro>
-	<xacro:loop links_qty="15" /> -->
+	<xacro:macro name="ball" params="d mass">
+		<link name='ball'>
+		<inertial>
+			<origin xyz="${d/2} 0 0 " />
+			<mass value="${mass}"/>
+			<inertia ixx="${mass* (d/2)**2 * (2/5)}" ixy="0.00" ixz="0.00" iyy="${mass* (d/2)**2 * (2/5)}" iyz="0.00" izz="${mass* (d/2)**2 * (2/5)}"/>
+		</inertial>
+		<collision name='collision'>
+			<origin xyz="${d/2} 0 0 "/>
+			<geometry>
+				<sphere radius="${d}"/>
+			</geometry>
+			<max_contacts>10</max_contacts>
+			<surface>
+				<contact>
+					<ode/>
+				</contact>
+				<bounce/>
+				<friction>
+					<torsional>
+						<ode/>
+					</torsional>
+					<ode/>
+				</friction>
+			</surface>
+		</collision>
+		<visual name='visual'>
+			<origin xyz="${d/2} 0 0 " />
+			<geometry>
+				<sphere radius="${d}"/>
+			</geometry>
+		</visual>
+		<self_collide>0</self_collide>
+		<enable_wind>0</enable_wind>
+		<kinematic>0</kinematic>
+	  </link>
+	</xacro:macro>
+	<!-- build chain links with base at the bottom usign the loop. build ball, attach to chain -->
+	<link name="chain_base"/>
+	<xacro:chain_link name="0" X="${link_length}" Y="0.01" Z="0.01" mass="0.001"/>
+		<joint name="0" type="fixed">
+			<origin xyz="0 0 0" rpy="0 0 0" />
+			<parent link="chain_base"/>
+			<child link="0"/>
+		</joint>
+	<xacro:link_gazebo name="0" />
+	<xacro:chain_loop i="${link_num}" />
+	<xacro:ball d="0.1" mass="1"/>
+	<xacro:link_gazebo name="ball"/>
+	<xacro:link_ball_joint name="ball" X="0" parent="${link_num}"/>
 </robot>

Commit message: prototyping cup and ball

File: jaco_gym/envs/assets/models/ball_and_cup/chain.urdf.xacro (robot description, xacro)
@@ -1,6 +1,8 @@
 <?xml version="1.0"?>
 <robot xmlns:xacro="http://www.ros.org/wiki/xacro" name="chain">
-	<xacro:property name="link_length" value="0.1" />
-	<xacro:property name="link_num" value="4"/>
+	<xacro:property name="link_length" value="0.025" />
+	<xacro:property name="link_yz" value="0.001"/>
+	<xacro:property name="link_num" value="20"/>
+	<xacro:property name="chain_link_mass" value="0.0001"/>
 	<xacro:macro name="chain_link" params="name X Y Z mass">
 		<link name="${name}">
@@ -25,42 +27,43 @@
 	</xacro:macro>
 	<xacro:macro name="link_ball_joint" params="name X parent">
-		<joint name="${name}_joint" type="continuous">
+		<joint name="${name}_x" type="continuous">
 			<origin xyz="${X} 0 0" rpy="0 0 0"/>
 			<parent link="${parent}"/>
-			<child link="${name}_junta1"/>
+			<child link="${name}_phi"/>
+			<axis xyz="1 0 0" />
+		</joint>
+		<link name="${name}_phi">
+			<inertial>
+			<mass value="0.0001" />
+			<inertia ixx="5.8083e-5" ixy="0" ixz="0" iyy="3.0833e-6" iyz="0" izz="5.9083e-5" />
+			</inertial>
+		</link>
+		<joint name="${name}_y" type="continuous">
+			<parent link="${name}_phi"/>
+			<child link="${name}_psi"/>
 			<axis xyz="0 1 0" />
 		</joint>
-		<link name="${name}_junta1">
+		<link name="${name}_psi">
 			<inertial>
-			<mass value="0.001" />
-			<inertia ixx="5.8083e-4" ixy="0" ixz="0" iyy="3.0833e-5" iyz="0" izz="5.9083e-4" />
+			<mass value="0.0001" />
+			<inertia ixx="5.8083e-5" ixy="0" ixz="0" iyy="3.0833e-6" iyz="0" izz="5.9083e-5" />
 			</inertial>
 		</link>
-		<joint name="${name}_joint2" type="continuous">
-			<parent link="${name}_junta1"/>
-			<child link="${name}_junta2"/>
+		<joint name="${name}_z" type="continuous">
+			<parent link="${name}_psi"/>
+			<child link="${name}"/>
 			<axis xyz="0 0 1" />
 		</joint>
-		<link name="${name}_junta2">
+		<!-- <link name="${name}_junta3">
 			<inertial>
-			<mass value="0.001" />
-			<inertia ixx="5.8083e-4" ixy="0" ixz="0" iyy="3.0833e-5" iyz="0" izz="5.9083e-4" />
+			<mass value="0.0001" />
+			<inertia ixx="5.8083e-5" ixy="0" ixz="0" iyy="3.0833e-6" iyz="0" izz="5.9083e-5" />
 			</inertial>
 		</link>
-		<joint name="${name}_joint3" type="continuous">
-			<parent link="${name}_junta1"/>
-			<child link="${name}_junta3"/>
-			<axis xyz="1 0 0" />
-		</joint>
-		<link name="${name}_junta3">
-			<inertial>
-			<mass value="0.001" />
-			<inertia ixx="5.8083e-4" ixy="0" ixz="0" iyy="3.0833e-5" iyz="0" izz="5.9083e-4" />
-			</inertial>
-		</link>
-		<joint name="${name}_jointfixed" type="fixed">
+		<joint name="${name}_jointfixed" type="continuous">
 			<parent link="${name}_junta3"/>
 			<child link="${name}"/>
-		</joint>
+			<axis xys="0 1 0"/>
+		</joint> -->
 	</xacro:macro>
 	<material name="Grey">
@@ -78,5 +81,5 @@
 	</xacro:macro>
 	<xacro:macro name="chain_loop" params="i">
-		<xacro:chain_link name="${link_num - i + 1}" X="${link_length}" Y="0.01" Z="0.01" mass="0.001"/>
+		<xacro:chain_link name="${link_num - i + 1}" X="${link_length}" Y="${link_yz}" Z="${link_yz}" mass="${chain_link_mass}"/>
 		<xacro:link_ball_joint name="${link_num - i + 1}" X="${link_length}" parent="${link_num - i}"/>
 		<xacro:link_gazebo name="${link_num - i + 1}"/>
@@ -87,42 +90,79 @@
 	<xacro:macro name="ball" params="d mass">
 		<link name='ball'>
-		<inertial>
-			<origin xyz="${d/2} 0 0 " />
-			<mass value="${mass}"/>
-			<inertia ixx="${mass* (d/2)**2 * (2/5)}" ixy="0.00" ixz="0.00" iyy="${mass* (d/2)**2 * (2/5)}" iyz="0.00" izz="${mass* (d/2)**2 * (2/5)}"/>
-		</inertial>
-		<collision name='collision'>
-			<origin xyz="${d/2} 0 0 "/>
-			<geometry>
-				<sphere radius="${d}"/>
-			</geometry>
-			<max_contacts>10</max_contacts>
-			<surface>
-				<contact>
-					<ode/>
-				</contact>
-				<bounce/>
-				<friction>
-					<torsional>
+			<inertial>
+				<origin xyz="${d} 0 0 " />
+				<mass value="${mass}"/>
+				<inertia ixx="${mass* (d/2)**2 * (2/5)}" ixy="0.00" ixz="0.00" iyy="${mass* (d/2)**2 * (2/5)}" iyz="0.00" izz="${mass* (d/2)**2 * (2/5)}"/>
+			</inertial>
+			<collision name='collision'>
+				<origin xyz="${d} 0 0 "/>
+				<geometry>
+					<sphere radius="${d}"/>
+				</geometry>
+				<max_contacts>10</max_contacts>
+				<surface>
+					<contact>
 						<ode/>
-					</torsional>
-					<ode/>
-				</friction>
-			</surface>
-		</collision>
-		<visual name='visual'>
-			<origin xyz="${d/2} 0 0 " />
-			<geometry>
-				<sphere radius="${d}"/>
-			</geometry>
-		</visual>
-		<self_collide>0</self_collide>
-		<enable_wind>0</enable_wind>
-		<kinematic>0</kinematic>
-	  </link>
+					</contact>
+					<bounce/>
+					<friction>
+						<torsional>
+							<ode/>
+						</torsional>
+						<ode/>
+					</friction>
+				</surface>
+			</collision>
+			<visual name='visual'>
+				<origin xyz="${d} 0 0 " />
+				<geometry>
+					<sphere radius="${d}"/>
+				</geometry>
+			</visual>
+			<self_collide>0</self_collide>
+			<enable_wind>0</enable_wind>
+			<kinematic>0</kinematic>
+	  	</link>
+	</xacro:macro>
+	<xacro:macro name="cup" params="mass">
+		<link name="cup">
+			<inertial>
+				<origin xyz="$0 0 0" />
+				<mass value="${mass}"/>
+				<inertia ixx="${mass * 0.282601}" ixy="${mass * 0.0056}" ixz="${mass * -0.000002}" iyy="${mass * 0.147524}" iyz="${mass * -0.007428}" izz="${mass * 0.276385}"/>
+			</inertial>
+			<collision name='collision'>
+				<origin xyz="0 0 0"/>
+				<geometry>
+					<mesh filename="file://../meshes/cup.dae"/>
+				</geometry>
+				<max_contacts>10</max_contacts>
+				<surface>
+					<contact>
+						<ode/>
+					</contact>
+					<bounce/>
+					<friction>
+						<torsional>
+							<ode/>
+						</torsional>
+						<ode/>
+					</friction>
+				</surface>
+			</collision>
+			<visual name='visual'>
+				<origin xyz="0 0 0" />
+				<geometry>
+					<mesh filename="file://../meshes/cup.dae"/>
+				</geometry>
+			</visual>
+			<self_collide>0</self_collide>
+			<enable_wind>0</enable_wind>
+			<kinematic>0</kinematic>
+	  	</link>
 	</xacro:macro>
 	<!-- build chain links with base at the bottom usign the loop. build ball, attach to chain -->
 	<link name="chain_base"/>
-	<xacro:chain_link name="0" X="${link_length}" Y="0.01" Z="0.01" mass="0.001"/>
+	<xacro:chain_link name="0" X="${link_length}" Y="${link_yz}" Z="${link_yz}" mass="0.001"/>
 		<joint name="0" type="fixed">
 			<origin xyz="0 0 0" rpy="0 0 0" />
@@ -132,6 +172,9 @@
 	<xacro:link_gazebo name="0" />
 	<xacro:chain_loop i="${link_num}" />
-	<xacro:ball d="0.1" mass="1"/>
+	<!-- <xacro:ball d="0.05" mass="1"/>
 	<xacro:link_gazebo name="ball"/>
-	<xacro:link_ball_joint name="ball" X="0" parent="${link_num}"/>
+	<xacro:link_ball_joint name="ball" X="${link_length}" parent="${link_num}"/> -->
+	<xacro:cup mass="1"/>
+	<xacro:link_gazebo name="cup"/>
+	<xacro:link_ball_joint name="cup" X="${link_length}" parent="${link_num}"/>
 </robot>
